File: bifrost.kicad_sch (KiCad schematic)
At the start: 24 parts, among them J1 USB4155-03-C_REVA, J2 HDMI_A_1.4, U1 TUSB322I, U2 HD3SS215IRTQR, U3 SN75DP139RGZR, U4 AP2112K-3.3, U5 TPS22918DBVR, U6 TPD4E05U06DQAR, U7 TPD4E05U06DQAR, U9 TPD8S300ARUKR

Commit message: ccaeuntahuntohu anouhe
Parts:
- added C10, C11, C12, C13, C14, C15, C16, C17, C18, C19, C8, C9: 0.1 uF, symbol Device:C_Small
- added C20: 0.1 uF, symbol Device:C
- added C21: 10 uF, symbol Device:C
- added R10, R6, R7, R8, R9: 10k, symbol Device:R_US
- added R11, R12: 2.2k, symbol Device:R_US
- added R13, R14, R15, R16, R17, R18, R19, R20: 22R, symbol Device:R_Small_US
- added R21, R22: 2.2K, symbol Device:R_Small_US
- added R23, R24, R25, R26: 1M, symbol Device:R_Small_US
- added R4: 1k, symbol Device:R_US
- added R5: 4.02k, symbol Device:R_US
Connections:
- net DB0+ is gone; now on net SSTXP2_F: U2.41 (DB0(p))
- net DB0- is gone; now on net SSTXN2_F: U2.40 (DB0(n))
- net DB1+ is gone; now on net SSRXP2_F: U2.38 (DB1(p))
- net DB1- is gone; now on net SSRXN2_F: U2.37 (DB1(n))
- net DB2+ is gone; now on net SSTXP1_F: U2.35 (DB2(p))
- net DB2- is gone; now on net SSTXN1_F: U2.34 (DB2(n))
- net DB3+ is gone; now on net SSRXP1_F: U2.32 (DB3(p))
- net DB3- is gone; now on net SSRXN1_F: U2.31 (DB3(n))
- net +3V3: now also U3.11 (VCC), U3.15 (VCC), U3.2 (VCC), U3.21 (VCC), U3.26 (VCC), U3.33 (VCC), U3.40 (VCC), U3.46 (VCC), C20.1, C21.1, R10.1, R11.2, R12.2, R21.1, R22.1, R6.2, R8.2
- net +5V: now also J2.18 (+5V)
- net DC0+: now also U3.39 (IN_D+), C12.1; no longer FL1.1, U2.2 (DC0(p))
- net DC0-: now also U3.38 (IN_D1-), C13.1; no longer FL1.4, U2.3 (DC0(n))
- net DC1+: now also U3.41 (IN_D2-), C15.1; no longer FL2.4, U2.5 (DC1(p))
- net DC1-: now also U3.42 (IN_D2+), C14.1; no longer FL2.1, U2.6 (DC1(n))
- net DC2+: now also U3.44 (IN_D3-), C17.1; no longer FL4.4, U2.8 (DC2(p))
- net DC2-: now also U3.45 (IN_D3+), C16.1; no longer FL4.1, U2.9 (DC2(n))
- net DC3+: now also U3.47 (IN_D4-), C19.1; no longer FL3.1, U2.11 (DC3(p))
- net DC3-: now also U3.48 (IN_D4+), C18.1; no longer FL3.4, U2.12 (DC3(n))
- net GND: now also J2.17 (GND), U2.1 (AUX_SEL), U3.1 (GND), U3.12 (GND), U3.18 (GND), U3.24 (GND), U3.27 (GND), U3.31 (GND), U3.36 (GND), U3.37 (GND), U3.43 (GND), U3.49 (EPAD), U3.5 (GND), C20.2, C21.2, R23.2, R24.2, R25.2, R26.2, R4.1, R5.2, R7.2, R9.1
- net SBU1: now also C11.2, C8.2
- net SBU2: now also C10.2, C9.2
- net HDMI_D1+: now reaches J2.1 (D2+)
- net HDMI_D1+: now also R14.2
- net HDMI_D4+: now reaches J2.10 (CK+)
- net HDMI_D4+: now also R20.2
- net HDMI_D4-: now reaches J2.12 (CK-)
- net HDMI_D4-: now also R19.2
- net HDMI_SCL: now reaches J2.15 (SCL)
- net HDMI_SCL: now also U3.28 (SCL_SINK), R11.1
- net HDMI_SDA: now reaches J2.16 (SDA)
- net HDMI_SDA: now also U3.29 (SDA_SINK), R12.1
- net HPD_SINK: now reaches J2.19 (HPD/HEAC-)
- net HPD_SINK: now also U3.30 (HPD_SINK), R4.2
- net HDMI_D1-: now reaches J2.3 (D2-)
- net HDMI_D1-: now also R13.2
- net HDMI_D2+: now reaches J2.4 (D1+)
- net HDMI_D2+: now also R16.2
- net HDMI_D2-: now reaches J2.6 (D1-)
- net HDMI_D2-: now also R15.2
- net HDMI_D3-: now reaches J2.7 (D0+)
- net HDMI_D3-: now also R17.2
- net HDMI_D3+: now reaches J2.9 (D0-)
- net HDMI_D3+: now also R18.2
- net AUX+: now reaches U2.13 (AUXC(p))
- net AUX-: now reaches U2.14 (AUXC(n))
- net at U2.15 (HPDC): now also U3.7 (HPD_SOURCE)
- net DDC_SCL: now reaches U2.18 (DDCCLK_C)
- net DDC_SCL: now also U3.9 (SCL_SOURCE), R21.2
- net at U2.22 (DDCCLK_B): now also R26.1
- net at U2.23 (DDCDAT_B): now also R25.1
- net at U2.24 (AUXB(p)): now also C10.1
- net at U2.25 (AUXB(n)): now also C11.1
- net DDC_SDA: now reaches U2.26 (DDCDAT_C)
- net DDC_SDA: now also U3.8 (SDA_SOURCE), R22.2
- net at U2.27 (DDCCLK_A): now also R23.1
- net at U2.28 (DDCDAT_A): now also R24.1
- net at U2.29 (AUXA(n)): now also C9.1
- net at U2.30 (AUXA(p)): now also C8.1
- net at U3.14 (OUT_D4-): now also R19.1
- net at U3.16 (OUT_D3+): now also R18.1
- net at U3.17 (OUT_D3-): now also R17.1
- net at U3.19 (OUT_D2+): now also R16.1
- net at U3.20 (OUT_D2-): now also R15.1
- net at U3.22 (OUT_D1+): now also R14.1
- net at U3.23 (OUT_D1-): now also R13.1
- net at U3.25 (OE_N): now also R7.1
- net at U3.3 (SRC): now also R6.1
- net at U3.32 (DDC_EN): now also R10.2
- net at U3.34 (HPDINV): now also R9.2
- net at U3.4 (I2C_EN): now also R8.1
- net at U3.6 (Vsadj): now also R5.1
- net DA0+ renamed SSTXP1_F
- net SSTXP1_F: now also FL1.1
- net DA0- renamed SSTXN1_F
- net SSTXN1_F: now also FL1.4
- net DA1+ renamed SSRXP1_F
- net SSRXP1_F: now also FL2.4
- net DA1- renamed SSRXN1_F
- net SSRXN1_F: now also FL2.1
- net DA2+ renamed SSTXP2_F
- net SSTXP2_F: now also FL4.4
- net DA2- renamed SSTXN2_F
- net SSTXN2_F: now also FL4.1
- net DA3+ renamed SSRXP2_F
- net SSRXP2_F: now also FL3.1
- net DA3- renamed SSRXN2_F
- net SSRXN2_F: now also FL3.4
- new net: C13.2, U2.3 (DC0(n))
- new net: C19.2, U2.11 (DC3(p))
- new net: C17.2, U2.8 (DC2(p))
- new net: C18.2, U2.12 (DC3(n))
- new net: C12.2, U2.2 (DC0(p))
- new net: C15.2, U2.5 (DC1(p))
- new net: C14.2, U2.6 (DC1(n))
- new net: C16.2, U2.9 (DC2(n))
- no-connect marks 20 -> 23
Other:
- note removed: "DP to HDMI Retimer"
- note removed: "Load Switch"
- moved on the sheet: C4, C5, C6, C7, FL3, FL4, J2, R1, R2, R3, U1, U2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

Commit message: schematic done? need to confirm some stuff
Parts:
- removed J2: HDMI_A_1.4, symbol Connector:HDMI_A_1.4
- removed R1, R2: 4.7k, symbol Device:R_US
- removed R10, R7, R8, R9: 10k, symbol Device:R_US
- removed R11, R12: 2.2k, symbol Device:R_US
- removed R13, R14, R15, R16, R17, R18, R19, R20: 22R, symbol Device:R_Small_US
- removed R4: 1k, symbol Device:R_US
- removed R5: 4.02k, symbol Device:R_US
- removed U3: SN75DP139RGZR, SN75DP139RGZR:RGZ48_4P1X4P1, symbol SN75DP139RGZR:SN75DP139RGZR
- removed U5: TPS22918DBVR, TPS22918DBVR:DBV6_TEX, symbol TPS22918DBVR:TPS22918DBVR
- added C22: 0.1 uF, symbol Device:C
- added R4: 1M, symbol Device:R_Small_US
- added R5: 5M, symbol Device:R_Small_US
- added U3: DisplayPort, symbol DISPLAYPORT-FEMALE:DisplayPort
- C20: value 0.1 uF -> 1 uF
- C21: value 10 uF -> 0.1 uF
- J1: footprint USB4155-03-C_REVA:GCT_USB4155-03-C_REVA -> USB-3-C-MALE:GCT_USB4155-03-C_REVA
- R21, R22: value 2.2K -> 100K
- R6: value 10k -> 1M
Connections:
- net +3V3: now also C22.1, U3.20 (DP_PWR); no longer C20.1, R22.1, R6.2
- net AUX+: now also R22.2, U3.15 (AUX_P)
- net AUX-: now also R21.2, U3.17 (AUX_N)
- net DC0+: now also U3.1 (D0_P)
- net DC0-: now also U3.3 (D0_N)
- net DC1+: now also U3.4 (D1_P)
- net DC1-: now also U3.6 (D1_N)
- net DC2+: now also U3.7 (D2_P)
- net DC2-: now also U3.9 (D2_N)
- net DC3+: now also U3.10 (D3_P)
- net DC3-: now also U3.12 (D3_N)
- net GND: now also R22.1, R6.2, U2.57 (PAD), C22.2, R4.1, R5.1, U3.19 (DP_PWR_RET); no longer U1.5 (ADDR)
- net at R6.1: now also C20.1, U3.11 (GND), U3.16 (GND), U3.2 (GND), U3.5 (GND), U3.8 (GND)
- net HPDC: now reaches U2.15 (HPDC)
- net HPDC: now also U3.18 (HPD)
- net DDC_SCL: no longer names the net of U2.18 (DDCCLK_C)
- net DDC_SCL: no longer R21.2
- net DDC_SDA: no longer names the net of U2.26 (DDCDAT_C)
- net DDC_SDA: no longer R22.2
- net SCL: no longer names the net of U1.8 (SCL/OUT2)
- net SDA: no longer names the net of U1.7 (SDA/OUT1)
- new net CFG1: R4.2, U3.13 (CFG1), U3.14 (CFG2)
- new net CFG2: R5.2
- no-connect marks 23 -> 29
Other:
- note added: "Orientation Mux"
- moved on the sheet: C10, C11, C12, C13, C14, C15, C16, C17, C18, C19, C4, C5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

Commit message: schematic done?
Parts:
- removed C4: 100 uF, symbol Device:C
- removed C5: 100 nF, symbol Device:C
- removed R3: 900k, symbol Device:R_US
- removed U1: TUSB322I, Package_DFN_QFN:Texas_X2QFN-12_1.6x1.6mm_P0.4mm, symbol Interface_USB:TUSB322I
- added C21, C22, C26, C27, C29, C32: 1 uF, symbol Device:C_Small
- added C23: 2.2 uF, symbol Device:C_Small
- added C24, C25: 1 uF, symbol Device:C
- added C28, C30: 27 pF, symbol Device:C_Small
- added C31: 0.1 uF, symbol Device:C_Small
- added R10: 200k, symbol Device:R_Small_US
- added R11, R12: 2.2k, symbol Device:R_Small_US
- added R13, R14: 47R, symbol Device:R_Small_US
- added unit 2 of U4
- added U5: 74LVC1G125, symbol 74xGxx:74LVC1G125
- added U6: MAX77958CEWV+T, MAX77958CEWV-T:21-100339_W302B3&plus_1_ADI, symbol MAX77958CEWV-T:MAX77958CEWV+T
- renumbered C20 to C1, C12 to C10, C15 to C11, C17 to C12, C19 to C13, C1 to C14, C3 to C15, C2 to C16, C8 to C17, C10 to C18, C9 to C19, C21 to C2, C11 to C20, C22 to C3, C13 to C4, C14 to C5, C16 to C6, C18 to C7, C7 to C8, C6 to C9, FL3 to FL2, FL4 to FL3, FL2 to FL4, R6 to R1, R4 to R2, R5 to R3, R21 to R4, R22 to R5, R26 to R6, R25 to R7, R23 to R8, R24 to R9, U3 to U1, U4 to U2, U2 to U3, U9 to U4, U6 to U7, U7 to U8
Connections:
- net +3V3: now also C26.1, C27.1, C32.1, R10.1, R11.1, R12.1, U4.10 (VPWR), U5.5 (VCC), U6.B1 (VIO1), U6.C1 (VIO2)
- net +5V: now also U2.3 (EN), C24.2, C25.2, C29.2, U6.A5 (VCIN), U6.A6 (VBUS), U6.B6 (VSS)
- net CC1: now also C30.1, U6.A3 (CC1)
- net CC2: now also C28.1, U6.A4 (CC2)
- net CFG1: no longer U1.14 (CFG2)
- net CFG2: now also U1.14 (CFG2)
- net DIR: now also U6.C4 (GPIO8)
- net GND: now also U1.SH, C21.1, C22.1, C23.2, C24.1, C25.1, C26.2, C27.2, C28.2, C29.1, C30.2, C31.2, C32.2, R13.2, R14.2, U4.13 (GND), U4.18 (GND), U4.21 (GND), U4.8 (GND), U5.1, U5.3 (GND), U6.C5 (GND_A), U6.D6 (GND_D)
- net HPDC: now also U5.4, U6.D3 (GPIO7); no longer U1.18 (HPD)
- new net: C31.1, U4.3 (VBIAS)
- new net: R13.1, U6.D1 (DN)
- new net: C22.2, U6.A2 (VDD1P1)
- new net: R14.1, U6.D2 (DP)
- new net: C21.2, U6.B5 (VDD1P8)
- new net: C23.1, U6.C6 (AVL)
- new net HPD_DP: U1.18 (HPD), U5.2
- new net INTB: R10.2, U6.A1 (INTB)
- new net SCL: R11.2, U6.B2 (SCL)
- new net SDA: R12.2, U6.B3 (SDA)
- no-connect marks 29 -> 35
Other:
- note added: "PD Controller"
- note removed: "CC Controller (orientation)"
- moved on the sheet: R2, R3

Commit message: testponits
Parts:
- added TP1: SCL, symbol Connector:TestPoint
- added TP2: SDA, symbol Connector:TestPoint
- added TP3: CC1, symbol Connector:TestPoint
- added TP4: CC2, symbol Connector:TestPoint
- added TP5: VBUS, symbol Connector:TestPoint
- added TP6: INTB, symbol Connector:TestPoint
- added TP7: DIR, symbol Connector:TestPoint
- added TP8: HPD, symbol Connector:TestPoint
- added TP9: 3V3, symbol Connector:TestPoint
Connections:
- net +3V3: now also TP9.1
- net +5V: now also TP5.1
- net CC1: now also TP3.1
- net CC2: now also TP4.1
- net DIR: now also TP7.1
- net HPDC: now also TP8.1
- net INTB: now also TP6.1
- net SCL: now also TP1.1
- net SDA: now also TP2.1

Commit message: thinking of re-layout
Parts:
- removed J1: USB4155-03-C_REVA, USB-3-C-MALE:GCT_USB4155-03-C_REVA, symbol USB-3-C-MALE:USB4155-03-C_REVA
- added USB1: ~, USB-3-C-MALE:USB-C-SMD_U261-241N-4BS2SS, symbol USB-3-C-MALE:U261-241N-4BS2SS
- C1, C10, C11, C12, C13, C14, C15, C16, C17, C18, C19, C2, C20, C21, C22, C24, C25, C26, C27, C28, C29, C3, C30, C31, C32, C4, C5, C6, C7, C8, C9: footprint (none) -> Capacitor_SMD:C_0603_1608Metric_Pad1.08x0.95mm_HandSolder
- C23: footprint (none) -> Capacitor_SMD:C_0805_2012Metric_Pad1.18x1.45mm_HandSolder
- R1, R10, R11, R12, R13, R14, R2, R3, R4, R5, R6, R7, R8, R9: footprint (none) -> Resistor_SMD:R_0603_1608Metric_Pad0.98x0.95mm_HandSolder
- TP1, TP2, TP3, TP4, TP5, TP6, TP7, TP8, TP9: footprint (none) -> TestPoint:TestPoint_Pad_D3.0mm
- U1: footprint (none) -> XDPF-0205-20S:DISPLAYPORT_FEMALE_XDPF-0205-20S
- U5: footprint (none) -> Package_TO_SOT_SMD:SOT-353_SC-70-5_Handsoldering
Connections:
- net +5V: now also USB1.A4 (VBUS), USB1.A9 (VBUS), USB1.B4 (VBUS), USB1.B9 (VBUS)
- net C_CC1: now also USB1.A5 (CC)
- net C_CC2: now also USB1.B5 (Vconn)
- net C_SBU1: now also USB1.A8 (SBU1)
- net C_SBU2: now also USB1.B8 (SBU2)
- net GND: now also USB1.25 (GND), USB1.26 (GND), USB1.A1 (GND), USB1.A12 (GND), USB1.B1 (GND), USB1.B12 (GND)
- net SSRXN1: now also USB1.B10 (RX1-)
- net SSRXN2: now also USB1.A10 (RX2-)
- net SSRXP1: now also USB1.B11 (RX1+)
- net SSRXP2: now also USB1.A11 (RX2+)
- net SSTXN1: now also USB1.A3 (TX1-)
- net SSTXN2: now also USB1.B3 (TX2-)
- net SSTXP1: now also USB1.A2 (TX1+)
- net SSTXP2: now also USB1.B2 (TX2+)
- net DC0_N: now reaches C4.2, U3.3 (DC0_N)
- net DC3_P: now reaches C13.2, U3.11 (DC3_P)
- net DC2_P: now reaches C12.2, U3.8 (DC2_P)
- net DC3_N: now reaches C7.2, U3.12 (DC3_N)
- net DC0_P: now reaches C10.2, U3.2 (DC0_P)
- net DC1_P: now reaches C11.2, U3.5 (DC1_P)
- net DC1_N: now reaches C5.2, U3.6 (DC1_N)
- net DC2_N: now reaches C6.2, U3.9 (DC2_N)
- net SSRXN1_F renamed F_SSRXN1
- net SSRXN2_F renamed F_SSRXN2
- net SSRXP1_F renamed F_SSRXP1
- net SSRXP2_F renamed F_SSRXP2
- net SSTXN1_F renamed F_SSTXN1
- net SSTXN2_F renamed F_SSTXN2
- net SSTXP1_F renamed F_SSTXP1
- net SSTXP2_F renamed F_SSTXP2
Other:
- moved on the sheet: C10, C11, C12, C13, C14, C15, C16, C4, C5, C6, C7, U2
